Commit message: 覆盖 Part 2 真机主链实现
- 基于最新 main 重建 aria、导航、视觉、安全与日志链\n- 新增 Docker/环境入口并统一 artifacts 输出\n- 修正定位、RGBD 配对与旧 ariaNode 构建冲突

File: src/p3at_description/urdf/pioneer.urdf.xacro (robot description, xacro)
@@ -197,4 +197,16 @@
   </joint>
   <link name="cam_optical_link"/>
+  <joint name="gps_joint" type="fixed">
+    <parent link="base_link"/>
+    <child link="gps_link"/>
+    <origin xyz="0 0 0.34" rpy="0 0 0"/>
+  </joint>
+  <link name="gps_link">
+    <inertial>
+      <mass value="1e-5"/>
+      <origin xyz="0 0 0"/>
+      <inertia ixx="1e-6" ixy="0" ixz="0" iyy="1e-6" iyz="0" izz="1e-6"/>
+    </inertial>
+  </link>
   <gazebo reference="laser_frame">
     <sensor name="front_lidar" type="gpu_lidar">
